File: circuit/hotbox.sch (KiCad schematic (older format))
At the start: 37 parts, among them IC1 ATMEGA48A-M, K1 CONN_3, P1 CONN_2, P2 CONN_5, P3 CONN_4, P4 CONN_3X2, U1 NCP1117ST33T3G, U2 OPTO-TRIAC, U3 BTA312Y-600C, U4 OPTO-TRANSISTOR4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

Commit message: 5x5cm version.
Parts:
- removed R12, R5, R6: R, Resistors_SMD:Resistor_SMD0805_ReflowWave, symbol R
- added RP1: 82R, symbol R_PACK4
- C2: value CP1 -> 220uF
- C3: value C -> 220uF
- C4: value C -> 0.1uF
- C5, C6: value C -> 12pF
- D1: value LED -> LED-orange
- D2: value LED -> LED-green
- D4: value LED -> LED-blue
- IC1: footprint SMD_Packages:TQFP32 -> SMD_Packages:QFN32
- R10: value R -> 330R
Connections:
- net labels added: zc
- wire segments 129 -> 136
- no-connect marks 16 -> 18
Other:
- moved on the sheet: D1, D2, D4, U4
Changed lines of the file:
@@
 F 0 "IC1" H 3350 4900 40  0000 L BNN
 F 1 "ATMEGA48A-M" H 4500 2250 40  0000 L BNN
-F 2 "SMD_Packages:TQFP32" H 4100 3650 30  0001 C CIN
+F 2 "SMD_Packages:QFN32" H 4100 3650 30  0001 C CIN
 F 3 "" H 4100 3650 60  0000 C CNN
 	1    4100 3650
@@
 P 6150 2950
 F 0 "C5" H 6150 3050 40  0000 L CNN
-F 1 "C" H 6156 2865 40  0000 L CNN
+F 1 "12pF" H 6156 2865 40  0000 L CNN
 F 2 "Capacitors_SMD:c_0805" H 6188 2800 30  0001 C CNN
 F 3 "" H 6150 2950 60  0000 C CNN
@@
 P 6150 3550
 F 0 "C6" H 6150 3650 40  0000 L CNN
-F 1 "C" H 6156 3465 40  0000 L CNN
+F 1 "12pF" H 6156 3465 40  0000 L CNN
 F 2 "Capacitors_SMD:c_0805" H 6188 3400 30  0001 C CNN
 F 3 "" H 6150 3550 60  0000 C CNN
@@
 F 3 "" H 10450 4200 60  0000 C CNN
 	1    10450 4200
-	1    0    0    -1
+	1    0    0    1
 $EndComp
 $Comp
 L LED D1
 U 1 1 5560D6DE
-P 7050 5050
-F 0 "D1" H 7050 5150 50  0000 C CNN
-F 1 "LED" H 7050 4950 50  0000 C CNN
-F 2 "LEDs:LED-0603" H 7050 5050 60  0001 C CNN
-F 3 "" H 7050 5050 60  0000 C CNN
-	1    7050 5050
+P 7050 5450
+F 0 "D1" H 7050 5550 50  0000 C CNN
+F 1 "LED-orange" H 7050 5350 50  0000 C CNN
+F 2 "LEDs:LED-0603" H 7050 5450 60  0001 C CNN
+F 3 "" H 7050 5450 60  0000 C CNN
+	1    7050 5450
 	1    0    0    -1
 $EndComp
@@
 L LED D2
 U 1 1 5560D704
-P 7050 5350
-F 0 "D2" H 7050 5450 50  0000 C CNN
-F 1 "LED" H 7050 5250 50  0000 C CNN
-F 2 "LEDs:LED-0603" H 7050 5350 60  0001 C CNN
-F 3 "" H 7050 5350 60  0000 C CNN
-	1    7050 5350
-	1    0    0    -1
-$EndComp
-$Comp
-L R R5
-U 1 1 5560D739
-P 6500 5050
-F 0 "R5" V 6580 5050 40  0000 C CNN
-F 1 "R" V 6507 5051 40  0000 C CNN
-F 2 "Resistors_SMD:Resistor_SMD0805_ReflowWave" V 6430 5050 30  0001 C CNN
-F 3 "" H 6500 5050 30  0000 C CNN
-	1    6500 5050
-	0    1    1    0
-$EndComp
-$Comp
-L R R6
-U 1 1 5560D74D
-P 6500 5350
-F 0 "R6" V 6580 5350 40  0000 C CNN
-F 1 "R" V 6507 5351 40  0000 C CNN
-F 2 "Resistors_SMD:Resistor_SMD0805_ReflowWave" V 6430 5350 30  0001 C CNN
-F 3 "" H 6500 5350 30  0000 C CNN
-	1    6500 5350
-	0    1    1    0
+P 7050 5200
+F 0 "D2" H 7050 5300 50  0000 C CNN
+F 1 "LED-green" H 7050 5100 50  0000 C CNN
+F 2 "LEDs:LED-0603" H 7050 5200 60  0001 C CNN
+F 3 "" H 7050 5200 60  0000 C CNN
+	1    7050 5200
+	1    0    0    -1
 $EndComp
 $Comp
@@
 NoConn ~ 5100 3700
 NoConn ~ 5100 4750
-NoConn ~ 5100 4850
 NoConn ~ 3200 4000
 NoConn ~ 3200 3900
@@
 P 2650 3500
 F 0 "C2" H 2700 3600 50  0000 L CNN
-F 1 "CP1" H 2700 3400 50  0000 L CNN
+F 1 "220uF" H 2700 3400 50  0000 L CNN
 F 2 "Capacitors_Tantalum_SMD:TantalC_SizeA_EIA-3216_Reflow" H 2650 3500 60  0001 C CNN
 F 3 "" H 2650 3500 60  0000 C CNN
@@
 P 3050 3350
 F 0 "C4" H 3050 3450 40  0000 L CNN
-F 1 "C" H 3056 3265 40  0000 L CNN
+F 1 "0.1uF" H 3056 3265 40  0000 L CNN
 F 2 "Capacitors_SMD:c_0805" H 3088 3200 30  0001 C CNN
 F 3 "" H 3050 3350 60  0000 C CNN
@@
 	0    1    1    0
 $EndComp
-Text Label 9850 4400 0    60   ~ 0
-load
 $Comp
 L NCP1117ST33T3G U1
@@
 P 7950 3900
 F 0 "R10" V 8030 3900 40  0000 C CNN
-F 1 "R" V 7957 3901 40  0000 C CNN
+F 1 "330R" V 7957 3901 40  0000 C CNN
 F 2 "Resistors_SMD:Resistor_SMD0805_HandSoldering" V 7880 3900 30  0001 C CNN
 F 3 "" H 7950 3900 30  0000 C CNN
@@
 P 2900 3050
 F 0 "C3" H 2900 3150 40  0000 L CNN
-F 1 "C" H 2906 2965 40  0000 L CNN
+F 1 "220uF" H 2906 2965 40  0000 L CNN
 F 2 "Capacitors_SMD:c_0805" H 2938 2900 30  0001 C CNN
 F 3 "" H 2900 3050 60  0000 C CNN
@@
 $EndComp
 $Comp
-L R R12
-U 1 1 55665CD3
-P 1850 3050
-F 0 "R12" V 1930 3050 40  0000 C CNN
-F 1 "R" V 1857 3051 40  0000 C CNN
-F 2 "Resistors_SMD:Resistor_SMD0805_ReflowWave" V 1780 3050 30  0001 C CNN
-F 3 "" H 1850 3050 30  0000 C CNN
-	1    1850 3050
-	1    0    0    -1
-$EndComp
-$Comp
 L LED D4
 U 1 1 55665CDE
-P 1850 3650
-F 0 "D4" H 1850 3750 50  0000 C CNN
-F 1 "LED" H 1850 3550 50  0000 C CNN
-F 2 "LEDs:LED-0603" H 1850 3650 60  0001 C CNN
-F 3 "" H 1850 3650 60  0000 C CNN
-	1    1850 3650
-	0    1    1    0
+P 7050 4950
+F 0 "D4" H 7050 5050 50  0000 C CNN
+F 1 "LED-blue" H 7050 4850 50  0000 C CNN
+F 2 "LEDs:LED-0603" H 7050 4950 60  0001 C CNN
+F 3 "" H 7050 4950 60  0000 C CNN
+	1    7050 4950
+	1    0    0    -1
 $EndComp
 $Sheet
@@
 F 3 "" H 6300 1500 60  0000 C CNN
 	1    6300 1500
-	1    0    0    -1
+	-1   0    0    -1
 $EndComp
 $Comp
@@
 TH2
 NoConn ~ 5100 2550
-NoConn ~ 5100 4350
 NoConn ~ 5100 4550
-Text Label 9900 4200 0    60   ~ 0
+$Comp
+L R_PACK4 RP1
+U 1 1 5568D5A7
+P 6550 5400
+F 0 "RP1" H 6550 5850 40  0000 C CNN
+F 1 "82R" H 6550 5350 40  0000 C CNN
+F 2 "" H 6550 5400 60  0000 C CNN
+F 3 "" H 6550 5400 60  0000 C CNN
+	1    6550 5400
+	1    0    0    -1
+$EndComp
+NoConn ~ 6750 5250
+NoConn ~ 6350 5250
+NoConn ~ 5100 4650
+Text Label 9850 4200 0    60   ~ 0
+load
+Text Label 9950 4300 0    60   ~ 0
 live
 Wire Wire Line
@@
 Connection ~ 3150 4850
 Wire Wire Line
-	3200 4750 3150 4750
-Wire Wire Line
 	5350 2950 5950 2950
 Wire Wire Line
@@
 	7950 1150 10600 1150
 Wire Wire Line
-	6050 5350 6250 5350
-Wire Wire Line
-	6750 5050 6850 5050
-Wire Wire Line
-	6850 5350 6750 5350
-Wire Wire Line
-	7250 4800 7250 5350
-Connection ~ 7250 5050
+	6750 5050 6850 4950
+Wire Wire Line
+	6850 5200 6750 5150
+Wire Wire Line
+	7250 4800 7250 5450
+Connection ~ 7250 4950
 Connection ~ 8550 3150
 Wire Wire Line
@@
 	3200 2550 3100 2550
 Connection ~ 3100 2650
-Wire Wire Line
-	1850 2650 3200 2650
 Connection ~ 3000 4850
 Wire Wire Line
@@
 Wire Wire Line
 	7750 4350 8050 4350
-Wire Wire Line
-	10100 4400 10100 4300
-Wire Wire Line
-	8550 4400 10100 4400
 Wire Wire Line
 	9200 3150 9050 3150
@@
 Wire Wire Line
 	3050 4050 3050 3550
-Wire Wire Line
-	1850 4050 3050 4050
 Connection ~ 2650 4050
 Wire Wire Line
@@
 	5100 4450 6250 4450
 Wire Wire Line
-	6250 4450 6250 5050
+	6250 4450 6250 5150
 Wire Wire Line
 	4950 5450 5450 5450
@@
 	6500 4800 7250 4800
 Wire Wire Line
-	7250 5050 7600 5050
-Wire Wire Line
-	7600 5050 7600 5100
+	7600 4950 7600 5100
 Wire Wire Line
 	7750 4350 7750 4550
 Wire Wire Line
-	3150 4650 3150 4850
-Wire Wire Line
 	3100 2550 3100 2650
-Wire Wire Line
-	3200 4650 3150 4650
-Connection ~ 3150 4750
 Wire Wire Line
 	2900 3250 2900 4050
@@
 	2900 2850 2900 2650
 Connection ~ 2900 2650
-Wire Wire Line
-	1850 3300 1850 3450
-Wire Wire Line
-	1850 3850 1850 4050
 Connection ~ 2350 4050
-Wire Wire Line
-	1850 2650 1850 2800
 Connection ~ 2350 2650
 Wire Wire Line
 	5100 1500 5100 1350
 Wire Wire Line
-	5100 1350 5650 1350
+	5100 1350 5700 1350
 Wire Wire Line
 	5650 1650 5650 2100
 Wire Wire Line
-	6900 1650 6900 2000
-Wire Wire Line
-	6900 2000 7050 2000
-Wire Wire Line
-	6900 1350 6900 900
-Wire Wire Line
-	6900 900  6950 900
-Wire Wire Line
 	2600 850  2600 950
 Wire Wire Line
@@
 Wire Wire Line
 	2750 1350 2550 1350
-Wire Wire Line
-	5100 2000 5100 2050
-Wire Wire Line
-	5100 2050 5500 2050
-Wire Wire Line
-	5500 2050 5500 3500
-Wire Wire Line
-	5500 3500 5100 3500
 Wire Wire Line
 	6500 4150 6500 3750
@@
 	5200 2850 5100 2850
 Wire Wire Line
-	5100 4650 6050 4650
-Wire Wire Line
-	6050 4650 6050 5350
+	6050 4350 6050 5350
 Wire Wire Line
 	9950 4100 9950 2850
 Connection ~ 9950 2850
 Wire Wire Line
-	10100 4200 9900 4200
-Wire Wire Line
 	8000 2000 7550 2000
 Wire Wire Line
 	9700 900  9700 2000
+Wire Wire Line
+	6850 5450 6750 5450
+Wire Wire Line
+	6750 5450 6750 5350
+Connection ~ 7250 5200
+Wire Wire Line
+	7600 4950 7250 4950
+Wire Wire Line
+	2350 4050 3050 4050
+Wire Wire Line
+	2350 2650 3200 2650
+Wire Wire Line
+	5400 5700 5400 5550
+Connection ~ 5400 5550
+Wire Wire Line
+	5650 1650 5700 1650
+Wire Wire Line
+	6950 900  6950 1350
+Wire Wire Line
+	6950 1650 6950 2000
+Wire Wire Line
+	6950 2000 7050 2000
+Connection ~ 4450 2050
+Connection ~ 5500 1350
+Wire Wire Line
+	5100 2050 4450 2050
+Wire Wire Line
+	5100 2000 5100 2050
+Wire Wire Line
+	3200 4650 3150 4650
+Wire Wire Line
+	3200 4750 3150 4750
+Connection ~ 3150 4750
+Wire Wire Line
+	3150 4650 3150 4850
+Wire Wire Line
+	5100 4350 6050 4350
+Wire Wire Line
+	6250 5150 6350 5150
+Wire Wire Line
+	6050 5350 6350 5350
+Wire Wire Line
+	6350 5050 6200 5050
+Wire Wire Line
+	6200 5050 6200 5700
+Wire Wire Line
+	6200 5700 5400 5700
+Wire Wire Line
+	9850 4400 9850 4200
+Wire Wire Line
+	9850 4200 10100 4200
+Connection ~ 9850 4400
+Wire Wire Line
+	8550 4400 9850 4400
+Wire Wire Line
+	10100 4300 9950 4300
+Wire Wire Line
+	5100 4850 5100 5250
+Wire Wire Line
+	5100 5250 4250 5250
+Wire Wire Line
+	5500 1000 4900 1000
+Text Label 4950 1000 0    60   ~ 0
+zc
+Text Label 4350 5250 0    60   ~ 0
+zc
+NoConn ~ 5100 3500
+Wire Wire Line
+	5500 1000 5500 1350
 $EndSCHEMATC

Commit message: Simplifid schematics removed snubber circuit (not necessary with BTA312Y).
Parts:
- removed C7, C8: C, Capacitors_SMD:c_1812, symbol C
- removed R11: R, Resistors_SMD:Resistor_SMD0805_ReflowWave, symbol R
- removed R9: R, Resistors_SMD:Resistor_SMD0805_HandSoldering, symbol R
- C2: footprint Capacitors_Tantalum_SMD:TantalC_SizeA_EIA-3216_Reflow -> Capacitors_Tantalum_SMD:TantalC_SizeC_EIA-6032_Reflow
- D3: footprint (none) -> custom:RECTIFIER_BRIDGE
- IC1: footprint SMD_Packages:QFN32 -> Housings_DFN_QFN:QFN-32-1EP_5x5mm_Pitch0.5mm
- P1: footprint (none) -> Socket_Strips:Socket_Strip_Straight_1x02
- P2: footprint (none) -> custom:CONN_AUDIO_JACK
- P4: footprint Socket_Strips:Socket_Strip_Straight_2x03 -> Pin_Headers:Pin_Header_Straight_2x03
- R10: footprint Resistors_SMD:Resistor_SMD0805_HandSoldering -> Resistors_SMD:R_0805
- RP1: footprint (none) -> Resistors_SMD:r_cat16-4
- U2: footprint SOT-4 -> custom:SOP-4
- U4: value OPTO-TRANSISTOR4 -> PC123; footprint DIP4F -> custom:DIP4F
Connections:
- wire segments 136 -> 142
Changed lines of the file:
@@
 LIBS:valves
 LIBS:hotbox-cache
-EELAYER 24 0
+EELAYER 25 0
 EELAYER END
 $Descr A4 11693 8268
@@
 F 0 "IC1" H 3350 4900 40  0000 L BNN
 F 1 "ATMEGA48A-M" H 4500 2250 40  0000 L BNN
-F 2 "SMD_Packages:QFN32" H 4100 3650 30  0001 C CIN
+F 2 "Housings_DFN_QFN:QFN-32-1EP_5x5mm_Pitch0.5mm" H 4100 3650 30  0001 C CIN
 F 3 "" H 4100 3650 60  0000 C CNN
 	1    4100 3650
@@
 $EndComp
 $Comp
-L R R9
-U 1 1 55611522
-P 7950 2850
-F 0 "R9" V 8030 2850 40  0000 C CNN
-F 1 "R" V 7957 2851 40  0000 C CNN
-F 2 "Resistors_SMD:Resistor_SMD0805_HandSoldering" V 7880 2850 30  0001 C CNN
-F 3 "" H 7950 2850 30  0000 C CNN
-	1    7950 2850
-	1    0    0    -1
-$EndComp
-$Comp
 L CONN_2 P1
 U 1 1 55626A8D
@@
 F 0 "P1" V 3050 1700 40  0000 C CNN
 F 1 "CONN_2" V 3150 1700 40  0000 C CNN
-F 2 "" H 3100 1700 60  0001 C CNN
+F 2 "Socket_Strips:Socket_Strip_Straight_1x02" H 3100 1700 60  0001 C CNN
 F 3 "" H 3100 1700 60  0000 C CNN
 	1    3100 1700
@@
 NoConn ~ 3200 3900
 $Comp
-L PWR_FLAG #FLG07
-U 1 1 55626C78
-P 2850 4800
-F 0 "#FLG07" H 2850 4895 30  0001 C CNN
-F 1 "PWR_FLAG" H 2850 4980 30  0000 C CNN
-F 2 "" H 2850 4800 60  0001 C CNN
-F 3 "" H 2850 4800 60  0000 C CNN
-	1    2850 4800
-	1    0    0    -1
-$EndComp
-$Comp
 L CP1 C2
 U 1 1 55626F50
@@
 F 0 "C2" H 2700 3600 50  0000 L CNN
 F 1 "220uF" H 2700 3400 50  0000 L CNN
-F 2 "Capacitors_Tantalum_SMD:TantalC_SizeA_EIA-3216_Reflow" H 2650 3500 60  0001 C CNN
+F 2 "Capacitors_Tantalum_SMD:TantalC_SizeC_EIA-6032_Reflow" H 2650 3500 60  0001 C CNN
 F 3 "" H 2650 3500 60  0000 C CNN
 	1    2650 3500
@@
 F 0 "P2" V 3100 1150 50  0000 C CNN
 F 1 "CONN_5" V 3200 1150 50  0000 C CNN
-F 2 "" H 3150 1150 60  0001 C CNN
+F 2 "custom:CONN_AUDIO_JACK" H 3150 1150 60  0001 C CNN
 F 3 "" H 3150 1150 60  0000 C CNN
 	1    3150 1150
@@
 $EndComp
 $Comp
-L R R11
-U 1 1 5564BA09
-P 8800 3150
-F 0 "R11" V 8880 3150 40  0000 C CNN
-F 1 "R" V 8807 3151 40  0000 C CNN
-F 2 "Resistors_SMD:Resistor_SMD0805_ReflowWave" V 8730 3150 30  0001 C CNN
-F 3 "" H 8800 3150 30  0000 C CNN
-	1    8800 3150
-	0    1    1    0
-$EndComp
-$Comp
-L C C8
-U 1 1 5564BA14
-P 9400 3150
-F 0 "C8" H 9400 3250 40  0000 L CNN
-F 1 "C" H 9406 3065 40  0000 L CNN
-F 2 "Capacitors_SMD:c_1812" H 9438 3000 30  0001 C CNN
-F 3 "" H 9400 3150 60  0000 C CNN
-	1    9400 3150
-	0    1    1    0
-$EndComp
-$Comp
 L NCP1117ST33T3G U1
 U 1 1 5564C108
@@
 $EndComp
 $Comp
-L GND #PWR08
+L GND #PWR07
 U 1 1 5564C11C
 P 4050 1900
-F 0 "#PWR08" H 4050 1900 30  0001 C CNN
+F 0 "#PWR07" H 4050 1900 30  0001 C CNN
 F 1 "GND" H 4050 1830 30  0001 C CNN
 F 2 "" H 4050 1900 60  0001 C CNN
@@
 	1    4050 1900
 	1    0    0    -1
-$EndComp
-$Comp
-L C C7
-U 1 1 5564C8F9
-P 9250 3750
-F 0 "C7" H 9250 3850 40  0000 L CNN
-F 1 "C" H 9256 3665 40  0000 L CNN
-F 2 "Capacitors_SMD:c_1812" H 9288 3600 30  0001 C CNN
-F 3 "" H 9250 3750 60  0000 C CNN
-	1    9250 3750
-	-1   0    0    1
 $EndComp
 $Comp
@@
 F 0 "R10" V 8030 3900 40  0000 C CNN
 F 1 "330R" V 7957 3901 40  0000 C CNN
-F 2 "Resistors_SMD:Resistor_SMD0805_HandSoldering" V 7880 3900 30  0001 C CNN
+F 2 "Resistors_SMD:R_0805" V 7880 3900 30  0001 C CNN
 F 3 "" H 7950 3900 30  0000 C CNN
 	1    7950 3900
@@
 F 0 "D3" H 8850 2050 70  0000 C CNN
 F 1 "BRIDGE" H 8850 1950 70  0000 C CNN
-F 2 "" H 8850 2000 60  0001 C CNN
+F 2 "custom:RECTIFIER_BRIDGE" H 8850 2000 60  0001 C CNN
 F 3 "" H 8850 2000 60  0000 C CNN
 	1    8850 2000
@@
 $EndComp
 $Comp
-L +3.3V #PWR09
+L +3.3V #PWR08
 U 1 1 5564D4F6
 P 6100 3850
-F 0 "#PWR09" H 6100 3810 30  0001 C CNN
+F 0 "#PWR08" H 6100 3810 30  0001 C CNN
 F 1 "+3.3V" H 6100 3960 30  0000 C CNN
 F 2 "" H 6100 3850 60  0001 C CNN
@@
 $EndComp
 $Comp
-L +3.3V #PWR010
+L +3.3V #PWR09
 U 1 1 5564D508
 P 4500 1200
-F 0 "#PWR010" H 4500 1160 30  0001 C CNN
+F 0 "#PWR09" H 4500 1160 30  0001 C CNN
 F 1 "+3.3V" H 4500 1310 30  0000 C CNN
 F 2 "" H 4500 1200 60  0001 C CNN
@@
 $EndComp
 $Comp
-L GND #PWR011
+L GND #PWR010
 U 1 1 5564DD38
 P 4950 5450
-F 0 "#PWR011" H 4950 5450 30  0001 C CNN
+F 0 "#PWR010" H 4950 5450 30  0001 C CNN
 F 1 "GND" H 4950 5380 30  0001 C CNN
 F 2 "" H 4950 5450 60  0001 C CNN
@@
 $EndComp
 $Comp
-L +3.3V #PWR012
+L +3.3V #PWR011
 U 1 1 5564DD4C
 P 5000 5550
-F 0 "#PWR012" H 5000 5510 30  0001 C CNN
+F 0 "#PWR011" H 5000 5510 30  0001 C CNN
 F 1 "+3.3V" H 5000 5660 30  0000 C CNN
 F 2 "" H 5000 5550 60  0001 C CNN
@@
 F 0 "P4" H 6700 2850 50  0000 C CNN
 F 1 "CONN_3X2" V 6700 2650 40  0000 C CNN
-F 2 "Socket_Strips:Socket_Strip_Straight_2x03" H 6700 2600 60  0001 C CNN
+F 2 "Pin_Headers:Pin_Header_Straight_2x03" H 6700 2600 60  0001 C CNN
 F 3 "" H 6700 2600 60  0000 C CNN
 	1    6700 2600
@@
 $EndComp
 $Comp
-L GND #PWR013
+L GND #PWR012
 U 1 1 5564E4A4
 P 7250 2550
-F 0 "#PWR013" H 7250 2550 30  0001 C CNN
+F 0 "#PWR012" H 7250 2550 30  0001 C CNN
 F 1 "GND" H 7250 2480 30  0001 C CNN
 F 2 "" H 7250 2550 60  0001 C CNN
@@
 $EndComp
 $Comp
-L +3.3V #PWR014
+L +3.3V #PWR013
 U 1 1 5564E4B8
 P 7250 2650
-F 0 "#PWR014" H 7250 2610 30  0001 C CNN
+F 0 "#PWR013" H 7250 2610 30  0001 C CNN
 F 1 "+3.3V" H 7250 2760 30  0000 C CNN
 F 2 "" H 7250 2650 60  0001 C CNN
@@
 F 0 "U2" H 7350 4650 60  0000 C CNN
 F 1 "OPTO-TRIAC" H 7250 4050 60  0000 C CNN
-F 2 "SOT-4" H 7150 4350 60  0001 C CNN
+F 2 "custom:SOP-4" H 7150 4350 60  0001 C CNN
 F 3 "" H 7150 4350 60  0000 C CNN
 	1    7150 4350
@@
 P 6300 1500
 F 0 "U4" H 6500 1750 60  0000 C CNN
-F 1 "OPTO-TRANSISTOR4" H 6300 1250 60  0000 C CNN
-F 2 "DIP4F" H 6300 1500 60  0001 C CNN
+F 1 "PC123" H 6300 1250 60  0000 C CNN
+F 2 "custom:DIP4F" H 6300 1500 60  0001 C CNN
 F 3 "" H 6300 1500 60  0000 C CNN
 	1    6300 1500
@@
 $EndComp
 $Comp
-L GND #PWR015
+L GND #PWR014
 U 1 1 55669CC6
 P 2600 850
-F 0 "#PWR015" H 2600 850 30  0001 C CNN
+F 0 "#PWR014" H 2600 850 30  0001 C CNN
 F 1 "GND" H 2600 780 30  0001 C CNN
 F 2 "" H 2600 850 60  0000 C CNN
@@
 F 0 "RP1" H 6550 5850 40  0000 C CNN
 F 1 "82R" H 6550 5350 40  0000 C CNN
-F 2 "" H 6550 5400 60  0000 C CNN
+F 2 "Resistors_SMD:r_cat16-4" H 6550 5400 60  0001 C CNN
 F 3 "" H 6550 5400 60  0000 C CNN
 	1    6550 5400
@@
 live
 Wire Wire Line
-	5450 3800 5100 3800
-Wire Wire Line
-	5100 3900 5450 3900
+	5100 3800 5550 3800
+Wire Wire Line
+	5100 3900 5550 3900
 Wire Wire Line
 	2600 6550 2600 6750
@@
 Connection ~ 3150 4850
 Wire Wire Line
-	5350 2950 5950 2950
-Wire Wire Line
-	5400 3550 5950 3550
+	5350 2950 6000 2950
+Wire Wire Line
+	5400 3550 6000 3550
 Wire Wire Line
 	5350 2950 5350 3150
@@
 	8850 2850 10650 2850
 Wire Wire Line
-	9700 900  7450 900
+	7350 900  9700 900
 Wire Wire Line
 	7950 1150 10600 1150
@@
 	7250 4800 7250 5450
 Connection ~ 7250 4950
-Connection ~ 8550 3150
-Wire Wire Line
-	8550 2600 8550 3750
-Wire Wire Line
-	7950 2600 7950 1150
 Connection ~ 8850 1150
 Wire Wire Line
@@
 Connection ~ 3000 4850
 Wire Wire Line
-	2850 4800 2850 4850
-Connection ~ 2850 4850
-Wire Wire Line
 	3050 3150 3200 3150
 Wire Wire Line
 	7750 4350 8050 4350
-Wire Wire Line
-	9200 3150 9050 3150
 Wire Wire Line
 	4050 1700 4050 1900
@@
 Connection ~ 4050 1800
 Wire Wire Line
-	2650 2150 2650 3300
-Wire Wire Line
-	2650 3700 2650 4850
-Wire Wire Line
-	7950 2600 8550 2600
-Wire Wire Line
-	7950 3100 7950 3650
-Wire Wire Line
-	7750 4150 7950 4150
-Wire Wire Line
-	9250 3950 9250 4400
-Connection ~ 9250 4400
-Wire Wire Line
-	9250 3550 7950 3550
-Connection ~ 7950 3550
-Wire Wire Line
-	9550 3150 9600 3150
-Wire Wire Line
-	9600 3150 9600 4400
+	2650 2150 2650 3350
+Wire Wire Line
+	2650 3650 2650 4850
+Wire Wire Line
+	7450 4150 7950 4150
 Connection ~ 9600 4400
 Connection ~ 2650 2650
 Wire Wire Line
-	3050 4050 3050 3550
+	3050 4050 3050 3500
 Connection ~ 2650 4050
 Wire Wire Line
@@
 	3100 2550 3100 2650
 Wire Wire Line
-	2900 3250 2900 4050
+	2900 4050 2900 3200
 Connection ~ 2900 4050
 Wire Wire Line
-	2350 2650 2350 3300
-Wire Wire Line
-	2350 3700 2350 4050
+	2350 2650 2350 3350
+Wire Wire Line
+	2350 3650 2350 4050
 Wire Wire Line
 	2900 2850 3200 2850
 Wire Wire Line
-	2900 2850 2900 2650
+	2900 2650 2900 2900
 Connection ~ 2900 2650
 Connection ~ 2350 4050
 Connection ~ 2350 2650
 Wire Wire Line
-	5100 1500 5100 1350
+	5100 1350 5100 1600
 Wire Wire Line
 	5100 1350 5700 1350
@@
 	2750 1350 2550 1350
 Wire Wire Line
-	6500 4150 6500 3750
+	6500 3750 6500 4250
 Wire Wire Line
 	6500 3750 7000 3750
@@
 Connection ~ 9950 2850
 Wire Wire Line
-	8000 2000 7550 2000
+	7450 2000 8000 2000
 Wire Wire Line
 	9700 900  9700 2000
@@
 	6950 1650 6950 2000
 Wire Wire Line
-	6950 2000 7050 2000
+	6950 2000 7150 2000
 Connection ~ 4450 2050
 Connection ~ 5500 1350
@@
 	5100 2050 4450 2050
 Wire Wire Line
-	5100 2000 5100 2050
+	5100 1900 5100 2050
 Wire Wire Line
 	3200 4650 3150 4650
@@
 Wire Wire Line
 	5500 1000 5500 1350
+Wire Wire Line
+	7050 900  6950 900
+Wire Wire Line
+	6300 2950 6350 2950
+Wire Wire Line
+	6350 3550 6300 3550
+Wire Wire Line
+	7000 3750 7000 3650
+Wire Wire Line
+	7000 3250 7000 3350
+Wire Wire Line
+	5950 3800 5850 3800
+Wire Wire Line
+	5950 3900 5850 3900
+Wire Wire Line
+	6500 4250 6850 4250
+Wire Wire Line
+	6850 4450 6500 4450
+Connection ~ 2900 2850
+Wire Wire Line
+	3050 3150 3050 3200
+Wire Wire Line
+	7950 4150 7950 4050
+Wire Wire Line
+	7450 4150 7450 4250
+Wire Wire Line
+	7450 4450 7450 4550
+Wire Wire Line
+	7450 4550 7750 4550
+Wire Wire Line
+	7950 1150 7950 3750
+Wire Wire Line
+	7950 3750 8550 3750
 $EndSCHEMATC
